File: DRV8428P-D11C-NEMA17.kicad_pcb (KiCad board)
At the start: 2 copper layers, 53.5 x 43 mm, 16 parts, among them J1 Conn_PinHeader_1x04_P2.54mm_H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, J2 Conn_PinHeader_2x02_P2.54mm_V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, J4 Conn_PinHeader_1x02_P2.54mm_H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, P1 Conn_USB_A_Plain, U1 MotorDriver_TI_DRV8428EPPWPR, U2 Regulator_Linear_LM3480-3.3V-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, U3 Microcontroller_ATSAMD11C14A-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

Commit message: Updated board
Other:
- board size 53.5 x 43 mm -> 53.2 x 43 mm
Changed lines of the file:
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@@
   (gr_circle (center 29.3 139.7) (end 30.8 139.7) (layer "Edge.Cuts") (width 1) (fill none))
   (gr_line (start 67 136.5) (end 63.5 133) (layer "Edge.Cuts") (width 1))
-  (gr_line (start 67 160.9) (end 67 172.5) (layer "Edge.Cuts") (width 1))
-  (gr_line (start 77.5 148.2) (end 77.5 160.9) (layer "Edge.Cuts") (width 1))
-  (gr_line (start 67 136.5) (end 66.9 147.9) (layer "Edge.Cuts") (width 1))
+  (gr_line (start 67 160.5) (end 67 172.5) (layer "Edge.Cuts") (width 1))
+  (gr_line (start 77.2 148.5) (end 77.2 160.5) (layer "Edge.Cuts") (width 1))
+  (gr_line (start 67 136.5) (end 67 148.499088) (layer "Edge.Cuts") (width 1))
   (gr_line (start 27.5 133) (end 63.5 133) (layer "Edge.Cuts") (width 1))
   (gr_circle (center 60.3 170.7) (end 61.8 170.7) (layer "Edge.Cuts") (width 1) (fill none))
   (gr_line (start 24 172.5) (end 24 136.5) (layer "Edge.Cuts") (width 1))
   (gr_line (start 67 172.5) (end 63.5 176) (layer "Edge.Cuts") (width 1))
-  (gr_line (start 67 160.9) (end 77.5 160.9) (layer "Edge.Cuts") (width 1))
+  (gr_line (start 67 160.5) (end 77.2 160.5) (layer "Edge.Cuts") (width 1))
   (gr_line (start 63.5 176) (end 27.5 176) (layer "Edge.Cuts") (width 1))
   (gr_line (start 27.5 133) (end 24 136.5) (layer "Edge.Cuts") (width 1))
@@
   (gr_circle (center 29.3 170.6) (end 30.8 170.6) (layer "Edge.Cuts") (width 1) (fill none))
   (gr_circle (center 60.3 139.7) (end 61.8 139.7) (layer "Edge.Cuts") (width 1) (fill none))
-  (gr_line (start 66.9 148.1) (end 77.4 148.1) (layer "Edge.Cuts") (width 1))
+  (gr_line (start 67 148.499088) (end 77.2 148.5) (layer "Edge.Cuts") (width 1))
   (gr_circle (center 45.5 154.5) (end 48.5 154.5) (layer "Edge.Cuts") (width 1) (fill none))
   (segment (start 29.2 166) (end 34.3 166) (width 0.3) (layer "F.Cu") (net 1))

Commit message: Updating the design
Parts:
- moved C3 4.24 mm to (53.0, 164.0)
- moved U2 3.07 mm to (51.9, 168.9)
- moved R4 2.72 mm to (61.4, 145.2)
- moved C2 1.90 mm to (40.2, 139.8)
Routing:
- net GND: track 228.5 -> 242.6 mm
- net +3V3: track 14.1 -> 18.0 mm
- net +5V: track 101.0 -> 97.7 mm
Other:
- board size 53.2 x 43 mm -> 52.7 x 42.3 mm
