File: DRV8428P-D11C-NEMA17.kicad_sch (KiCad schematic)
At the start: 16 parts, among them J1 Conn_PinHeader_1x04_P2.54mm_H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, J2 Conn_PinHeader_2x02_P2.54mm_V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, J4 Conn_PinHeader_1x02_P2.54mm_H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, P1 Conn_USB_A_Plain, U1 MotorDriver_TI_DRV8428EPPWPR, U2 Regulator_Linear_LM3480-3.3V-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, U3 Microcontroller_ATSAMD11C14A-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

Commit message: Updating the design
Parts:
- U1: value MotorDriver_TI_DRV8428EPPWPR -> MotorDriver_TI_DRV8428PPWPR
Changed lines of the file:
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@@
     (in_bom yes) (on_board yes)
     (property "Reference" "U1" (id 0) (at 58.42 101.3206 0))
-    (property "Value" "MotorDriver_TI_DRV8428EPPWPR" (id 1) (at 58.42 103.632 0))
+    (property "Value" "MotorDriver_TI_DRV8428PPWPR" (id 1) (at 58.42 103.632 0))
     (property "Footprint" "fab:HTSSOP-16" (id 2) (at 58.42 81.28 0)
       (effects (font (size 1.27 1.27)) hide)
@@
   (symbol (lib_id "fab:Power_GND") (at 54.61 33.02 180) (unit 1)
     (in_bom yes) (on_board yes)
-    (property "Reference" "#PWR?" (id 0) (at 54.61 26.67 0)
+    (property "Reference" "#PWR0107" (id 0) (at 54.61 26.67 0)
       (effects (font (size 1.27 1.27)) hide)
     )
@@
       (reference "#PWR0106") (unit 1) (value "Power_GND") (footprint "")
     )
+    (path "/426ed018-908d-4928-9655-74918ceb5cf7"
+      (reference "#PWR0107") (unit 1) (value "Power_GND") (footprint "")
+    )
     (path "/070f5656-44a4-40d9-ad2b-45e70b1de6b0"
       (reference "#PWR0108") (unit 1) (value "Power_+5V") (footprint "")
@@
       (reference "#PWR0118") (unit 1) (value "Power_+5V") (footprint "")
     )
-    (path "/426ed018-908d-4928-9655-74918ceb5cf7"
-      (reference "#PWR?") (unit 1) (value "Power_GND") (footprint "")
-    )
     (path "/00000000-0000-0000-0000-000061e9e5f9"
       (reference "C1") (unit 1) (value "1uF") (footprint "fab:C_1206")
@@
     )
     (path "/00000000-0000-0000-0000-000061e96a34"
-      (reference "U1") (unit 1) (value "MotorDriver_TI_DRV8428EPPWPR") (footprint "fab:HTSSOP-16")
+      (reference "U1") (unit 1) (value "MotorDriver_TI_DRV8428PPWPR") (footprint "fab:HTSSOP-16")
     )
     (path "/00000000-0000-0000-0000-000061ea1d48"
